File: esp_module_basic/vers2_cheaper.kicad_pcb (KiCad board)
At the start: 2 copper layers, 19 parts, among them P1 CONN_01X4, P2 CONN_01X15, P3 CONN_01X15

Commit message: Edgecuts and silkscreen layers
Other:
- board outline added: 49 x 90.1 mm
- board text added: "DEFCON 25"
- board text added: "MRB"
